File: Hardware/Production/SparkFun_MicroMod_Function_SARA-R5-Panel.brd (EAGLE design)
At the start: 127.2 x 155.4 mm, 768 parts, among them J1 MICROMOD_FUNCTION_STANDARD, J10 U.FL, J11 MICROMOD_FUNCTION_STANDARD, J13 U.FL, J14 NANO_SIM, J15 U.FL, J16 MICROMOD_FUNCTION_STANDARD, J18 U.FL, J19 NANO_SIM, J2 U.FL, J20 U.FL, J21 MICROMOD_FUNCTION_STANDARD, J23 U.FL, J24 NANO_SIM, J25 U.FL, J26 MICROMOD_FUNCTION_STANDARD, J28 U.FL, J29 NANO_SIM, J30 U.FL, J4 U.FL, J5 MICROMOD_FUNCTION_STANDARD, J7 U.FL, J8 NANO_SIM, J9 NANO_SIM, Q1 310mA/60V/1.6Ω, Q10 310mA/60V/1.6Ω, Q11 310mA/60V/1.6Ω, Q12 310mA/60V/1.6Ω, Q13 310mA/60V/1.6Ω, Q14 310mA/60V/1.6Ω, Q15 310mA/60V/1.6Ω, Q16 310mA/60V/1.6Ω, Q17 310mA/60V/1.6Ω, Q18 310mA/60V/1.6Ω, Q19 310mA/60V/1.6Ω, Q2 310mA/60V/1.6Ω, Q20 310mA/60V/1.6Ω, Q21 310mA/60V/1.6Ω, Q22 310mA/60V/1.6Ω, Q23 310mA/60V/1.6Ω, Q24 310mA/60V/1.6Ω, Q3 310mA/60V/1.6Ω, Q4 310mA/60V/1.6Ω, Q5 310mA/60V/1.6Ω, Q6 310mA/60V/1.6Ω, Q7 310mA/60V/1.6Ω, Q8 310mA/60V/1.6Ω, Q9 310mA/60V/1.6Ω, U1 SARA-R510M8S, U10 SARA-R510M8S, U11 74HC1G04, U12 3.3V, U13 EEPROM, U14 AP7361C-33FGE, U15 74HC1G04, U16 SN74AVC4T774PW, U17 SARA-R510M8S, U18 3.3V, U19 EEPROM, U2 SN74AVC4T774PW, U20 AP7361C-33FGE, U21 74HC1G04, U22 SN74AVC4T774PW, U23 SARA-R510M8S, U24 3.3V, U25 EEPROM, U26 AP7361C-33FGE, U27 74HC1G04, U28 SN74AVC4T774PW, U29 SARA-R510M8S, U3 3.3V, U30 3.3V, U31 EEPROM, U32 AP7361C-33FGE, U33 74HC1G04, U34 SN74AVC4T774PW, U35 SARA-R510M8S, U36 3.3V, U4 EEPROM, U5 AP7361C-33FGE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

Commit message: v11 production panel and gerbers
Parts:
- R102, R126, R16, R33, R54, R78: value 100k -> DNP
- R113, R137, R29, R46, R65, R89: value 330 -> 100
Connections:
- net CTS: no longer R32.2
- net CTS1: no longer R22.2
- net CTS2: no longer R60.2
- net CTS3: no longer R84.2
- net CTS4: no longer R108.2
- net CTS5: no longer R132.2
- net GND: now also U2.7; no longer U2.8
- net GND1: now also U9.7; no longer U9.8
- net GND2: now also U16.7; no longer U16.8
- net GND3: now also U22.7; no longer U22.8
- net GND4: now also U28.7; no longer U28.8
- net GND5: now also U34.7; no longer U34.8
- net RTS: now also R32.2
- net RTS1: now also R22.2
- net RTS2: now also R60.2
- net RTS3: now also R84.2
- net RTS4: now also R108.2
- net RTS5: now also R132.2
- net VCCIO: now also U2.8; no longer U2.7
- net VCCIO1: now also U9.8; no longer U9.7
- net VCCIO2: now also U16.8; no longer U16.7
- net VCCIO3: now also U22.8; no longer U22.7
- net VCCIO4: now also U28.8; no longer U28.7
- net VCCIO5: now also U34.8; no longer U34.7
Routing:
- net RTS1: track 15.0 -> 16.8 mm, vias 1 -> 2
- net RTS: track 15.0 -> 16.8 mm, vias 1 -> 2
- net RTS2: track 15.0 -> 16.8 mm, vias 1 -> 2
- net RTS4: track 15.0 -> 16.8 mm, vias 1 -> 2
- net RTS3: track 15.0 -> 16.8 mm, vias 1 -> 2
- net RTS5: track 15.0 -> 16.8 mm, vias 1 -> 2
- net VCCIO4: track 105.6 -> 106.3 mm
- net VCCIO: track 105.6 -> 106.3 mm
- net VCCIO5: track 105.6 -> 106.3 mm
- net VCCIO3: track 105.6 -> 106.3 mm
- net VCCIO2: track 105.6 -> 106.3 mm
- net VCCIO1: track 105.6 -> 106.3 mm
- net CTS1: track 18.1 -> 17.8 mm, vias 2 -> 1
- net CTS: track 18.1 -> 17.8 mm, vias 2 -> 1
- net CTS5: track 18.1 -> 17.8 mm, vias 2 -> 1
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Other:
- board text added: "v11"
- board text removed: "v10"

Commit message: On LED changed to Red (DIO-17976)
Parts:
- D12, D17, D26, D36, D46, D56: value GREEN -> RED
Changed lines of the file:
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@@
 <layer number="25" name="tNames" color="7" fill="1" visible="no" active="yes"/>
 <layer number="26" name="bNames" color="7" fill="1" visible="no" active="yes"/>
-<layer number="27" name="tValues" color="7" fill="1" visible="no" active="yes"/>
+<layer number="27" name="tValues" color="7" fill="1" visible="yes" active="yes"/>
 <layer number="28" name="bValues" color="7" fill="1" visible="no" active="yes"/>
 <layer number="29" name="tStop" color="7" fill="3" visible="no" active="yes"/>
@@
 <layer number="98" name="Guide" color="6" fill="1" visible="no" active="no"/>
 <layer number="99" name="SpiceOrder" color="7" fill="1" visible="no" active="no"/>
-<layer number="100" name="Muster" color="7" fill="1" visible="no" active="yes"/>
+<layer number="100" name="Muster" color="7" fill="1" visible="yes" active="yes"/>
 <layer number="101" name="Patch_Top" color="12" fill="4" visible="no" active="no"/>
 <layer number="102" name="Vscore" color="7" fill="1" visible="no" active="no"/>
@@
 <attribute name="VALUE" value="240" x="0.581659375" y="20.8169" size="0.6096" layer="27" font="vector" ratio="20" rot="R270" align="top-center"/>
 </element>
-<element name="D17" library="SparkFun-LED" package="LED-0603" value="GREEN" x="4.345" y="17.272" smashed="yes" rot="R90">
+<element name="D17" library="SparkFun-LED" package="LED-0603" value="RED" x="4.345" y="17.272" smashed="yes" rot="R90">
 <attribute name="NAME" x="3.71" y="17.272" size="0.6096" layer="25" font="vector" ratio="20" rot="R90" align="bottom-center"/>
-<attribute name="PROD_ID" value="DIO-00821" x="158.015" y="-71.628" size="1.778" layer="27" font="vector" ratio="15" rot="R90" display="off"/>
+<attribute name="PROD_ID" value="DIO-17976" x="158.015" y="-71.628" size="1.778" layer="27" font="vector" ratio="15" rot="R90" display="off"/>
 <attribute name="VALUE" x="4.98" y="17.272" size="0.6096" layer="27" font="vector" ratio="20" rot="R90" align="top-center"/>
 </element>
@@
 <attribute name="VALUE" value="240" x="38.580059375" y="20.8169" size="0.6096" layer="27" font="vector" ratio="20" rot="R270" align="top-center"/>
 </element>
-<element name="D12" library="SparkFun-LED" package="LED-0603" value="GREEN" x="42.3434" y="17.272" smashed="yes" rot="R90">
+<element name="D12" library="SparkFun-LED" package="LED-0603" value="RED" x="42.3434" y="17.272" smashed="yes" rot="R90">
 <attribute name="NAME" x="41.7084" y="17.272" size="0.6096" layer="25" font="vector" ratio="20" rot="R90" align="bottom-center"/>
-<attribute name="PROD_ID" value="DIO-00821" x="196.0134" y="-71.628" size="1.778" layer="27" font="vector" ratio="15" rot="R90" display="off"/>
+<attribute name="PROD_ID" value="DIO-17976" x="196.0134" y="-71.628" size="1.778" layer="27" font="vector" ratio="15" rot="R90" display="off"/>
 <attribute name="VALUE" x="42.9784" y="17.272" size="0.6096" layer="27" font="vector" ratio="20" rot="R90" align="top-center"/>
 </element>
@@
 <attribute name="VALUE" value="240" x="76.578459375" y="20.8169" size="0.6096" layer="27" font="vector" ratio="20" rot="R270" align="top-center"/>
 </element>
-<element name="D26" library="SparkFun-LED" package="LED-0603" value="GREEN" x="80.3418" y="17.272" smashed="yes" rot="R90">
+<element name="D26" library="SparkFun-LED" package="LED-0603" value="RED" x="80.3418" y="17.272" smashed="yes" rot="R90">
 <attribute name="NAME" x="79.7068" y="17.272" size="0.6096" layer="25" font="vector" ratio="20" rot="R90" align="bottom-center"/>
-<attribute name="PROD_ID" value="DIO-00821" x="234.0118" y="-71.628" size="1.778" layer="27" font="vector" ratio="15" rot="R90" display="off"/>
+<attribute name="PROD_ID" value="DIO-17976" x="234.0118" y="-71.628" size="1.778" layer="27" font="vector" ratio="15" rot="R90" display="off"/>
 <attribute name="VALUE" x="80.9768" y="17.272" size="0.6096" layer="27" font="vector" ratio="20" rot="R90" align="top-center"/>
 </element>
@@
 <attribute name="VALUE" value="240" x="36.908740625" y="115.532840625" size="0.6096" layer="27" font="vector" ratio="20" rot="R90" align="top-center"/>
 </element>
-<element name="D36" library="SparkFun-LED" package="LED-0603" value="GREEN" x="33.1454" y="119.077740625" smashed="yes" rot="R270">
+<element name="D36" library="SparkFun-LED" package="LED-0603" value="RED" x="33.1454" y="119.077740625" smashed="yes" rot="R270">
 <attribute name="NAME" x="33.7804" y="119.077740625" size="0.6096" layer="25" font="vector" ratio="20" rot="R270" align="bottom-center"/>
-<attribute name="PROD_ID" value="DIO-00821" x="-120.5246" y="207.977740625" size="1.778" layer="27" font="vector" ratio="15" rot="R270" display="off"/>
+<attribute name="PROD_ID" value="DIO-17976" x="-120.5246" y="207.977740625" size="1.778" layer="27" font="vector" ratio="15" rot="R270" display="off"/>
 <attribute name="VALUE" x="32.5104" y="119.077740625" size="0.6096" layer="27" font="vector" ratio="20" rot="R270" align="top-center"/>
 </element>
@@
 <attribute name="VALUE" value="240" x="74.907140625" y="115.532840625" size="0.6096" layer="27" font="vector" ratio="20" rot="R90" align="top-center"/>
 </element>
-<element name="D46" library="SparkFun-LED" package="LED-0603" value="GREEN" x="71.1438" y="119.077740625" smashed="yes" rot="R270">
+<element name="D46" library="SparkFun-LED" package="LED-0603" value="RED" x="71.1438" y="119.077740625" smashed="yes" rot="R270">
 <attribute name="NAME" x="71.7788" y="119.077740625" size="0.6096" layer="25" font="vector" ratio="20" rot="R270" align="bottom-center"/>
-<attribute name="PROD_ID" value="DIO-00821" x="-82.5262" y="207.977740625" size="1.778" layer="27" font="vector" ratio="15" rot="R270" display="off"/>
+<attribute name="PROD_ID" value="DIO-17976" x="-82.5262" y="207.977740625" size="1.778" layer="27" font="vector" ratio="15" rot="R270" display="off"/>
 <attribute name="VALUE" x="70.5088" y="119.077740625" size="0.6096" layer="27" font="vector" ratio="20" rot="R270" align="top-center"/>
 </element>
@@
 <attribute name="VALUE" value="240" x="112.905540625" y="115.532840625" size="0.6096" layer="27" font="vector" ratio="20" rot="R90" align="top-center"/>
 </element>
-<element name="D56" library="SparkFun-LED" package="LED-0603" value="GREEN" x="109.1422" y="119.077740625" smashed="yes" rot="R270">
+<element name="D56" library="SparkFun-LED" package="LED-0603" value="RED" x="109.1422" y="119.077740625" smashed="yes" rot="R270">
 <attribute name="NAME" x="109.7772" y="119.077740625" size="0.6096" layer="25" font="vector" ratio="20" rot="R270" align="bottom-center"/>
-<attribute name="PROD_ID" value="DIO-00821" x="-44.5278" y="207.977740625" size="1.778" layer="27" font="vector" ratio="15" rot="R270" display="off"/>
+<attribute name="PROD_ID" value="DIO-17976" x="-44.5278" y="207.977740625" size="1.778" layer="27" font="vector" ratio="15" rot="R270" display="off"/>
 <attribute name="VALUE" x="108.5072" y="119.077740625" size="0.6096" layer="27" font="vector" ratio="20" rot="R270" align="top-center"/>
 </element>
